File: schematic.kicad_sch (KiCad schematic)
At the start: 43 parts, among them J1 Current Testing, J2 USB4105-GF-A, J3 Conn_01x04_Pin, J4 Conn_01x04_Pin, SW1 Boot, SW3 Boot, SW4 Boot, SW5 Boot, SW6 Boot, U1 ESP32-S3-MINI-1-N8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

Commit message: uploaded Schematic / PCB / any other needed files
Parts:
- removed C3, C4: 1u, Capacitor_SMD:C_0402_1005Metric, symbol Device:C
- removed D4: SP0503BAHTG, ESD Prot:SOT143, symbol ESD Prot:SP0503BAHTG
- removed J2: USB4105-GF-A, Connector_USB:USB_C_Receptacle_GCT_USB4105-xx-A_16P_TopMnt_Horizontal, symbol USB C:USB4105-GF-A
- removed U3: LP5907MFX-3.3, Package_TO_SOT_SMD:SOT-23-5, symbol 3V3Reg:LP5907MFX-3.3
- added C8, C9: 1u, Capacitor_SMD:C_0805_2012Metric, symbol Device:C
- added D10: SP0503BAHTG, Package_TO_SOT_SMD:SOT-143, symbol ESD Prot:SP0503BAHTG
- added D9: LED, LED_SMD:LED_0805_2012Metric, symbol Device:LED
- added J5: USB_C_Receptacle_USB2.0_16P, Connector_USB:USB_C_Receptacle_GCT_USB4105-xx-A_16P_TopMnt_Horizontal, symbol Connector:USB_C_Receptacle_USB2.0_16P
- added R13: R, Resistor_SMD:R_0805_2012Metric, symbol Device:R
- added U6: LP5907MFX-3.3, Package_TO_SOT_SMD:SOT-23-5, symbol Regulator_Linear:LP5907MFX-3.3
- BT1: footprint Library:Battery -> Connector_PinSocket_2.54mm:PinSocket_1x02_P2.54mm_Vertical
- C1, C2, C5, C6, C7: footprint Capacitor_SMD:C_0402_1005Metric -> Capacitor_SMD:C_0805_2012Metric
- D3: footprint LED_SMD:LED_0603_1608Metric -> LED_SMD:LED_0805_2012Metric
- D5, D6, D7, D8: footprint (none) -> LED_SMD:LED_0805_2012Metric
- R1, R12, R2, R3, R4, R5, R6, R7: footprint Resistor_SMD:R_0402_1005Metric -> Resistor_SMD:R_0805_2012Metric
- R10, R11, R8, R9: footprint (none) -> Resistor_SMD:R_0805_2012Metric
- S1: footprint slide switch v3:SW_JS102011SAQN -> Button_Switch_SMD:SW_SPDT_CK_JS102011SAQN
- U1: footprint MyFootprints:XCVR_ESP32-S3-MINI-1-N8 -> esp-s3-mini-1:XCVR_ESP32-S3-MINI-1-N8
- U5: footprint (none) -> Custom_Lora:Lora_Adafruit
Connections:
- net +3V3: now also U5.1 (Vin), C9.1, U6.5 (OUT)
- net +5V: now also D10.4, J5.A4 (VBUS), J5.A9 (VBUS), J5.B4 (VBUS), J5.B9 (VBUS)
- net CC1: no longer R5.2
- net CC2: no longer R6.2
- net DN: now also D10.3, J5.A7 (D-), J5.B7 (D-)
- net DP: now also D10.2, J5.A6 (D+), J5.B6 (D+)
- net GND: now also R7.2, U5.2 (GND), C8.2, C9.2, D10.1, J5.A1 (GND), J5.A12 (GND), J5.B1 (GND), J5.B12 (GND), R13.2, U6.2 (GND); no longer R7.1
- net RX: now also U1.40 (RXD0)
- net TX: now also U1.39 (TXD0)
- net VDD: now also C8.1, U6.1 (IN), U6.3 (EN)
- net at U1.28 (IO33): no longer D7.2 (A)
- net at U1.6 (IO2): no longer SW5.2
- net LED_4: now reaches U1.16 (IO12)
- net LED_4: now also D8.2 (A)
- net LED_5: now reaches U1.17 (IO13)
- net LED_5: now also D9.2 (A)
- net at U1.25 (IO21): no longer D5.2 (A)
- net at U1.26 (IO26): no longer D6.2 (A)
- net LORA_G5: now reaches U1.27 (IO47)
- net LORA_G5: now also U5.14 (G5)
- net LORA_CS: now reaches U1.29 (IO34)
- net LORA_CS: now also U5.8 (CS); no longer D8.2 (A)
- net LORA_MOSI: now reaches U1.31 (IO35)
- net LORA_MOSI: now also U5.7 (MOSI)
- net LORA_SCK: now reaches U1.32 (IO36)
- net LORA_SCK: now also U5.5 (SCK)
- net LORA_MISO: now reaches U1.33 (IO37)
- net LORA_MISO: now also U5.6 (MISO)
- net LORA_EN: now reaches U1.34 (IO38)
- net LORA_EN: now also U5.3 (EN)
- net LORA_GO: now reaches U1.35 (IO39)
- net LORA_GO: now also U5.4 (G0)
- net LORA_RST: now reaches U1.36 (IO40)
- net LORA_RST: now also U5.9 (RST)
- net LORA_G1: now reaches U1.37 (IO41)
- net LORA_G1: now also U5.10 (G1)
- net LORA_G2: now reaches U1.38 (IO42)
- net LORA_G2: now also U5.11 (G2)
- net LORA_G3: now reaches U1.41 (IO45)
- net LORA_G3: now also U5.12 (G3)
- net LORA_G4: now reaches U1.44 (IO46)
- net LORA_G4: now also U5.13 (G4)
- net at U1.5 (IO1): no longer SW4.2
- net at U1.7 (IO3): no longer SW6.2
- net G renamed LED_2
- net LED_2: now also D6.2 (A); no longer U5.14 (G4)
- net G1 renamed BTN_1
- net BTN_1: now also SW4.2; no longer U5.10 (G1)
- net G2 renamed BTN_2
- net BTN_2: now also SW5.2; no longer U5.11 (G2)
- net G3 renamed BTN_3
- net BTN_3: now also SW6.2; no longer U5.12 (G3)
- net G4 renamed LED_1
- net LED_1: now also D5.2 (A); no longer U5.13 (G4)
- net LoRaEN renamed LED_3
- net LED_3: now also D7.2 (A); no longer U5.3 (EN)
- net SCL renamed OLED_SCL
- net SDA renamed OLED_SDA
- new net: J5.B5 (CC2), R5.2
- new net: D9.1 (K), R13.1
- new net: J5.S1 (SHIELD), R7.1
- new net: J5.A5 (CC1), R6.2
- no-connect marks 19 -> 4
Other:
- note added: "5/1/2024"
- note added: "COM BTNS"
- note added: "DIRECTIONAL LEDS"
- note added: "MICROCONTROLLER"
- note added: "WaveLink Schemat 1.0"
- moved on the sheet: BT1, C5, C6, C7, D1, D2, D3, D5, D6, D7, D8, J1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
